File: kicad-source/main-board/antenna-analyzer.kicad_pcb (KiCad board)
At the start: 2 copper layers, 80 x 60 mm, 32 parts, among them M1 100uA, P1 5k LIN, SW1 RS1010-2Pole-4Pos

Commit message: Add files via upload
Parts:
- added H6: ~, User_Global_Library:mousebites-metric-5, F.Cu at (83.5, 111.0)
- H5: footprint User_Global_Library:mousebites-metric-5 -> User_Global_Library:mousebites-metric-5-trackgap
- moved H7 5.50 mm to (69.5, 111.0)
Connections:
- J2 pad 1: GND2 -> GND
- J3 pad 1: GND2 -> GND
- J4 pad 1: unconnected-(J4-Pin_1-Pad1) -> GND
- M1 pad 1: GND2 -> GND
- R8 pad 2: GND2 -> GND
Routing:
- net GND: track 0.00 -> 56.1 mm
- net GND2: track 42.8 -> 0.00 mm
Other:
- outline, holes or cut-outs redrawn
