File: kicad-source/main-board/antenna-analyzer.kicad_sch (KiCad schematic)
At the start: 32 parts, among them M1 100uA, P1 5k LIN, SW1 RS1010-2Pole-4Pos

Commit message: Add files via upload
Parts:
- added H6: ~, User_Global_Library:mousebites-metric-5, symbol User_Global_Symbol_Library:mousebites
- H5: footprint User_Global_Library:mousebites-metric-5 -> User_Global_Library:mousebites-metric-5-trackgap
Connections:
- net GND2 is gone; now on net GND: J2.1 (Pin_1), J3.1 (Pin_1), M1.1 (-), R8.2
- net GND: now also J4.1 (Pin_1)
- no-connect marks 8 -> 7
